File: v1_schematic.brd (EAGLE design)
At the start: 100 x 80 mm, 212 parts, among them IC1 PCA82C250, IC2 FT232RL, IC3 SP3223EBP, IC4 MAX481CPA, IC5 LM2576T, Q1 25MHz, Q2 32.768kHz, Q3 2N2222A, T1 ST02-3.5MM, T3 2N2222, T4 2N2222, T5 2N2222, T6 2N2222, T7 2N2222, U1 ON_SEMICONDUCTOR_NCP1117ST33T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, U2 ON_SEMICONDUCTOR_NCP1117ST50T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, X1 MINI-USB-32005-201, X10 PC817SW, X11 PC817SW, X12 PC817SW, X13 PC817SW, X14 PC817SW, X15 PC817SW, X16 PC817SW, X17 PC817SW, X18 PC817SW, X19 PC817SW, X20 PC817SW, X21 PC817SW, X22 PC817SW, X23 PC817SW, X24 PC817SW, X6 SDBMF, X7 5566-8, X8 5566-8, X9 PC817SW

Commit message: Board
- Added dimension
Parts:
- moved U$1 137.6 mm to (-2.54, 30.5)
- moved C15 74.1 mm to (-213.4, 114.3)
- moved C18 74.1 mm to (-97.8, 120.7)
- moved C25 74.1 mm to (-142.2, 120.7)
- moved C30 74.1 mm to (-174.0, 120.7)
- moved C43 74.1 mm to (-163.8, 44.5)
- moved C45 74.1 mm to (-177.8, 44.5)
- moved C6 74.1 mm to (-181.6, 114.3)
- moved C7 74.1 mm to (-188.0, 114.3)
- moved DIR1 74.1 mm to (-146.1, 144.8)
- moved DIR13 74.1 mm to (-97.8, 151.1)
- moved DIR6 74.1 mm to (-184.2, 144.8)
- moved DIR7 74.1 mm to (-191.8, 144.8)
- moved IC1 74.1 mm to (-191.8, 43.2)
- moved IC2 74.1 mm to (-188.0, 96.5)
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Other:
- board size 100 x 80 mm -> 150.8 x 88.9 mm
