File: v1 blocks/v1_schematic.brd (EAGLE design)
At the start: 150.8 x 88.9 mm, 212 parts, among them IC1 PCA82C250, IC2 FT232RL, IC3 SP3223EBP, IC4 MAX481CPA, IC5 LM2576T, Q1 25MHz, Q2 32.768kHz, Q3 2N2222A, T1 ST02-3.5MM, T3 2N2222, T4 2N2222, T5 2N2222, T6 2N2222, T7 2N2222, U1 ON_SEMICONDUCTOR_NCP1117ST33T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, U2 ON_SEMICONDUCTOR_NCP1117ST50T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, X1 MINI-USB-32005-201, X10 PC817SW, X11 PC817SW, X12 PC817SW, X13 PC817SW, X14 PC817SW, X15 PC817SW, X16 PC817SW, X17 PC817SW, X18 PC817SW, X19 PC817SW, X20 PC817SW, X21 PC817SW, X22 PC817SW, X23 PC817SW, X24 PC817SW, X6 5566-20, X7 5566-8, X8 5566-8, X9 PC817SW

Commit message: V2
Created new layout template
Parts:
- removed T3, T4, T5, T6, T7: 2N2222, transistor-neu-to92:TO18
- added Q4, Q5, Q6, Q7, Q8: (no value), semicon-smd-ipc:SOT23
- moved S2 305.0 mm to (46.7, 38.9)
- moved S3 304.8 mm to (24.9, 56.6)
- moved C14 304.4 mm to (54.7, 39.4), turned to 270 degrees
- moved R7 292.3 mm to (25.0, 48.3), turned to 90 degrees
- moved L2 274.2 mm to (14.2, 27.1)
- moved C16 267.6 mm to (38.7, 45.0), turned to 90 degrees
- moved R11 265.6 mm to (12.1, 30.9), turned to 180 degrees
- moved C15 263.7 mm to (33.3, 21.0), turned to 270 degrees
- moved C51 256.1 mm to (10.7, 19.9), turned to 180 degrees
- moved R28 246.4 mm to (-4.32, 20.8), turned to 270 degrees
- moved R6 243.7 mm to (16.3, 14.9), turned to 180 degrees
- moved R5 241.5 mm to (16.4, 10.9), turned to 180 degrees
- moved LED3 239.4 mm to (10.3, 14.9)
- moved LED2 236.7 mm to (10.3, 10.9)
- moved R22 217.7 mm to (0.89, 20.8), turned to 90 degrees
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Connections:
- net GND: now also Q8.2; no longer T7.1
- net GND2: now also Q8.3; no longer T7.3
- net N$49: now also Q4.1; no longer T3.2
- net N$51: now also Q5.1; no longer T4.2
- net N$52: now also Q6.1; no longer T5.2
- net N$54: now also Q7.1; no longer T6.2
- net N$55: now also Q8.1; no longer T7.2
- net R1IN: now also Q7.2; no longer T6.1
- net R1IN_: now also Q7.3; no longer T6.3
- net R2IN: now also Q5.2; no longer T4.1
- net R2IN_: now also Q5.3; no longer T4.3
- net T1OUT: now also Q6.2; no longer T5.1
- net T1OUT_: now also Q6.3; no longer T5.3
- net T2OUT: now also Q4.2; no longer T3.1
- net T2OUT_: now also Q4.3; no longer T3.3
Other:
- board size 150.8 x 88.9 mm -> 166.2 x 99.4 mm
