File: v1.1 blocks/schema_mpb1_1.sch (EAGLE design)
At the start: 81 parts, among them Q3 25MHz, Q4 32.768kHz, U1 NCP1117ST33T3G, U2 NCP1117ST50T3G, X1 PCI-60-POS-145167, X2 PCI-60-POS-145167, X3 PCI-60-POS-145167, X5 POWERSUPPLY_DC21MMX, X7 5566-20

Commit message: UPDATE
Updated design for Main board and I/O
- Reduced form factor, boards will be interconnected using ribbon cable connectors on 20-pin headers
Parts:
- removed H5, H6, H7, H8: MOUNT-PAD-ROUND3.2, holes:MOUNT-PAD-ROUND3.2
- removed J1: (no value), SparkFun-Connectors:CONN_03
- removed Q3: 25MHz, special:XTAL/S
- removed Q4: 32.768kHz, special:XTAL/S
- removed R16, R17, R18, R19, R20: 10K, rcl:R-EU_R0805
- removed S4, S6: STS121PC04, switches:STS121PC04
- removed S5: DTS-6, switch-tact:DTS-6
- removed X1, X3: PCI-60-POS-145167, con-amp:PCI-60-POS-145167
- removed X7: 5566-20, con-molex:5566-20
- added 3V3, B0, B1: (no value), jumper:SJ2W
- added C6: 1uF, SmartPrj:C-EU0603-RND
- added C7: 100nF, SmartPrj:C-EU0603-RND
- added CTS, RTS: (no value), jumper:SJ
- added F1: 500mA, adafruit:PTCFUSE-1812
- added I/O, JP3, JP4, JP5, JP6, SERIAL: (no value), pinhead-2:PINHD-2X10_2.00
- added IC1: CP2102, silabs-2:CP2102
- added JP1: (no value), pinhead:PINHD-1X6
- added JTAG: (no value), pinhead-2:PINHD-2X05_2.00
- added L1: (no value), rcl:L-EUL1812
- added Q1: 8M, crystal:CRYSTALHC49UP
- added Q2: 32.768kHz, crystal:CRYSTALHC49UP
- added R4, R5: 10K, rcl:R-EU_R0603
- added R7: 4k7, resistor:R-EU_R0603
- added R8, R9: 10k, resistor:R-EU_R0603
- added RESET: SWITCH-MOMENTARY-2SMD-1101NE, SparkFun-Electromechanical:SWITCH-MOMENTARY-2SMD-1101NE
- added SJ1: JUMPER-PAD-3-NO, SparkFun-Passives:JUMPER-PAD-3-NO
- C10, C11, C12, C13, C42, C43, C44, C45, C46, C47, C48, C49, C50, C51, C52, C53, C54, C55, C56, C57, C58, C59, C60, C61, C62, C63, C64, C65, C66, C67, C68, C69: device resistor:C-EUC0805 -> resistor:C-EUC0603
- R13, R14, R15, R21: device resistor:R-EU_R0805 -> resistor:R-EU_R0603
- X2: value PCI-60-POS-145167 -> PN61729-S; device con-amp:PCI-60-POS-145167 -> con-berg:PN61729-S
Connections:
- removed net UART4_RX: U$2.PA1
- removed net UART4_TX: U$2.PA0
- removed net USART3_RX: U$2.PB11
- removed net USART3_TX: U$2.PB10
- new net N$11: IC1.RI, JP1.3
- new net N$21: IC1.!SUSPEND, JP1.2, R9.2
- new net N$22: I/O.17
- new net N$23: I/O.19
- new net N$24: JTAG.8
- new net N$25: JTAG.10
- new net N$26: IC1.SUSPEND, JP1.1
- new net N$27: IC1.DTR, JP1.5
- new net N$32: IC1.DSR, JP1.6
- new net N$41: CTS.1, IC1.RTS
- new net N$44: IC1.CTS, RTS.1
- new net N$49: I/O.18
- new net N$5: B1.2, R4.1
- new net N$50: I/O.20
- new net N$6: B0.2, R5.1
- new net N$8: IC1.!RST, R7.2, R8.2
- new net PA2: U$2.PA2
- new net PA3: U$2.PA3
- new net RX3: SERIAL.6, U$2.PB11
- new net RX4: SERIAL.8, U$2.PA1
- new net TX3: SERIAL.5, U$2.PB10
- new net TX4: SERIAL.7, U$2.PA0
- new net VUSB2: F1.1, SJ1.1
- net +12V: now also 3V3.3; no longer J1.1
- net +3V3: now also B0.1, B1.1, C7.1, IC1.VDD, JTAG.1; no longer S4.3, S6.3, X7-1.S, X7-2.S
- net +5V: now also C6.1, IC1.REGIN, IC1.VBUS, SJ1.2; no longer J1.3
- net BOOT0: now also R5.2; no longer R17.1
- net BOOT1: now also R4.2; no longer R16.2
- net GND: now also B0.3, B1.3, C6.2, C7.2, IC1.GND, IC1.GND@EXP, IC1.GND@M, R8.1, R9.1, RESET.2, X2.4, X2.S1, X2.S2, X6-2.KL; no longer R18.2, R19.2, R20.2, S4.1, S5.1, S5.2, S6.1, X6-1.KL, X7-10.S, X7-12.S, X7-14.S, X7-16.S, X7-18.S, X7-20.S, X7-4.S, X7-6.S, X7-8.S
- net N$10: now also Q2.2; no longer Q4.2
- net N$12: now also Q2.1; no longer Q4.1
- net N$13: now also IC1.D-, X2.2; no longer R16.1, S4.2
- net N$14: now also IC1.D+, X2.3; no longer C42.2, S5.3, S5.4
- net N$15: now also JTAG.9; no longer R17.2, S6.2
- net N$17: now also L1.2, R7.1, X2.1; no longer R18.1, X7-11.S
- net N$18: now also F1.2, L1.1; no longer R19.1, X7-17.S
- net N$19: now also IC1.DCD, JP1.4; no longer R20.1, X7-19.S
- net N$45: now also 3V3.2; no longer J1.2
- net N$9: now also Q1.2; no longer Q3.2
- net NRF_SCK: now also JTAG.6; no longer X7-13.S
- net PE0: now also I/O.1
- net PE1: now also I/O.2
- net PE10: now also I/O.11
- net PE11: now also I/O.12
- net PE12: now also I/O.13
- net PE13: now also I/O.14
- net PE14: now also I/O.15
- net PE15: now also I/O.16
- net PE2: now also I/O.3
- net PE3: now also I/O.4
- net PE4: now also I/O.5
- net PE5: now also I/O.6
- net PE6: now also I/O.7
- net PE7: now also I/O.8
- net PE8: now also I/O.9
- net PE9: now also I/O.10
- net PH1: now also Q1.1; no longer Q3.1
- net REG_5V: now also 3V3.1, SJ1.3
- net RESET: now also C42.2, RESET.1
- net RESET#: now also JTAG.7; no longer X7-15.S
- net TCK/SWCLK: now also JTAG.5; no longer X7-9.S
- net TDI: now also JTAG.3; no longer X7-5.S
- net TMS/SWDIO: now also JTAG.4; no longer X7-7.S
- net TRST: now also JTAG.2; no longer X7-3.S
- net USART2_CTS: now also CTS.2
- net USART2_RTS: now also RTS.2
- net USART2_RX: now also IC1.TXD; no longer U$2.PA3
- net USART2_TX: now also IC1.RXD; no longer U$2.PA2
- net VIN: now also X6-1.KL; no longer X6-2.KL
Other:
- note added: "(RX0)"
- note added: "(TX0)"
- note added: "USB-UART Bridge"
- note removed: "TDO/SWO"
- note removed: "TRST"
- moved on the sheet: C10, C11, C12, C13, C42, C43, C44, C45, C46, C47, C48, C49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

Commit message: Routing
First draft of routing tracks for main board
Parts:
- removed C57, C58, C59, C60, C61, C62, C63: 100nF, resistor:C-EUC0603
- removed C64, C67: 4.7uF, resistor:C-EUC0603
- removed JP3, JP5, JP6: (no value), pinhead-2:PINHD-2X10_2.00
- added COM: (no value), pinhead-2:PINHD-2X10_2.54
- I/O, JP4, SERIAL: device pinhead-2:PINHD-2X10_2.00 -> pinhead-2:PINHD-2X10_2.54
Connections:
- removed net +3V3: B0.1, B1.1, C45.1, C46.1, C47.1, C48.1, C49.1, C50.1, C51.1, C52.1, C53.1, C54.1, C55.1, C56.1, C57.1, C58.1, C59.1, C60.1, C61.1, C62.1, C63.1, C64.1, C67.1, C7.1, IC1.VDD, JTAG.1, L3.1, U$2.VDD, U$2.VDD1, U$2.VDD2, U$2.VDD3, U$2.VDD4, U$2.VDD5
- removed net N$22: I/O.17
- removed net N$23: I/O.19
- removed net N$49: I/O.18
- removed net N$50: I/O.20
- removed net PA10: U$2.PA10
- removed net PA2: U$2.PA2
- removed net PA3: U$2.PA3
- removed net PA8: U$2.PA8
- removed net PA9: U$2.PA9
- removed net PB9: U$2.PB9
- removed net R1OUT: U$2.PB0
- removed net T1IN: U$2.PB1
- new net PB12: U$2.PB12
- new net PB13: U$2.PB13
- new net PB14: U$2.PB14
- new net PB15: U$2.PB15
- new net RX1: SERIAL.2, U$2.PB1
- new net RX2: SERIAL.4, U$2.PA3
- new net RX5: SERIAL.10, U$2.PA9
- new net RX6: SERIAL.12, U$2.PB9
- new net TX1: SERIAL.1, U$2.PB0
- new net TX2: SERIAL.3, U$2.PA2
- new net TX5: SERIAL.9, U$2.PA8
- new net TX6: SERIAL.11, U$2.PA10
- net +12V: now also I/O.18
- net +5V: now also COM.15, COM.16, I/O.19, SERIAL.15, SERIAL.16
- net 3.3V: now also B0.1, B1.1, C45.1, C46.1, C47.1, C48.1, C49.1, C50.1, C51.1, C52.1, C53.1, C54.1, C55.1, C56.1, C7.1, COM.19, COM.20, I/O.20, IC1.VDD, JTAG.1, L3.1, SERIAL.19, SERIAL.20, U$2.VDD, U$2.VDD1, U$2.VDD2, U$2.VDD3, U$2.VDD4, U$2.VDD5
- net CAN1_TX: now also COM.5, COM.6
- net ETH_MISO: now also COM.3; no longer U$2.PB14
- net ETH_MOSI: now also COM.4; no longer U$2.PB15
- net ETH_SCK: now also COM.2; no longer U$2.PB13
- net ETH_SS: now also COM.1; no longer U$2.PB12
- net GND: now also COM.13, COM.14, COM.17, COM.18, I/O.15, I/O.16, SERIAL.13, SERIAL.14, SERIAL.17, SERIAL.18; no longer C57.2, C58.2, C59.2, C60.2, C61.2, C62.2, C63.2, C64.2, C67.2
- net NRF_CE: now also COM.10
- net NRF_CS: now also COM.11
- net NRF_IRQ: now also COM.12
- net NRF_MISO: now also COM.9
- net NRF_MOSI: now also COM.8
- net NRF_SCK: now also COM.7
- net PE14: no longer I/O.15
- net PE15: no longer I/O.16
- net VIN: now also I/O.17

Commit message: Power Tracks
Routed main power tracks for Main board PCB
Parts:
- removed JP4: (no value), pinhead-2:PINHD-2X10_2.54
Connections:
- removed net PB14: U$2.PB14
- removed net PB15: U$2.PB15
- new net USB_OTG_HS_DM: COM.13, U$2.PB14
- new net USB_OTG_HS_DP: COM.14, U$2.PB15
- net +12V: now also I/O.20; no longer I/O.18
- net 3.3V: now also I/O.17; no longer I/O.20
- net GND: no longer COM.13, COM.14
- net VIN: now also I/O.18; no longer I/O.17
Changed lines of the file:
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@@
 <part name="SERIAL" library="pinhead-2" deviceset="PINHD-2X10" device="_2.54"/>
 <part name="COM" library="pinhead-2" deviceset="PINHD-2X10" device="_2.54"/>
-<part name="JP4" library="pinhead-2" deviceset="PINHD-2X10" device="_2.54"/>
 <part name="IC1" library="silabs-2" deviceset="CP210*" device="" technology="2"/>
 <part name="X2" library="con-berg" deviceset="PN61729-S" device=""/>
@@
 <instance part="SERIAL" gate="A" x="55.88" y="193.04"/>
 <instance part="COM" gate="A" x="55.88" y="160.02"/>
-<instance part="JP4" gate="A" x="55.88" y="124.46"/>
 <instance part="IC1" gate="G$1" x="154.94" y="78.74"/>
 <instance part="X2" gate="G$1" x="96.52" y="83.82" rot="MR0"/>
@@
 </segment>
 <segment>
-<pinref part="COM" gate="A" pin="13"/>
-<wire x1="53.34" y1="154.94" x2="43.18" y2="154.94" width="0.1524" layer="91"/>
-<label x="43.18" y="154.94" size="1.27" layer="95" rot="R180" xref="yes"/>
-</segment>
-<segment>
-<pinref part="COM" gate="A" pin="14"/>
-<wire x1="60.96" y1="154.94" x2="73.66" y2="154.94" width="0.1524" layer="91"/>
-<label x="73.66" y="154.94" size="1.27" layer="95" xref="yes"/>
-</segment>
-<segment>
 <pinref part="I/O" gate="A" pin="15"/>
 <wire x1="53.34" y1="218.44" x2="43.18" y2="218.44" width="0.1524" layer="91"/>
@@
 </segment>
 <segment>
-<pinref part="I/O" gate="A" pin="20"/>
-<wire x1="60.96" y1="213.36" x2="71.12" y2="213.36" width="0.1524" layer="91"/>
-<label x="81.28" y="213.36" size="1.778" layer="95" xref="yes"/>
-</segment>
-<segment>
 <pinref part="SERIAL" gate="A" pin="20"/>
 <wire x1="60.96" y1="180.34" x2="71.12" y2="180.34" width="0.1524" layer="91"/>
@@
 <pinref part="C54" gate="G$1" pin="1"/>
 <junction x="116.078" y="172.974"/>
+</segment>
+<segment>
+<pinref part="I/O" gate="A" pin="17"/>
+<wire x1="53.34" y1="215.9" x2="43.18" y2="215.9" width="0.1524" layer="91"/>
+<label x="43.18" y="215.9" size="1.778" layer="95" rot="R180" xref="yes"/>
 </segment>
 </net>
@@
 <net name="VIN" class="1">
 <segment>
-<pinref part="I/O" gate="A" pin="17"/>
-<wire x1="53.34" y1="215.9" x2="43.18" y2="215.9" width="0.1524" layer="91"/>
-<label x="43.18" y="215.9" size="1.778" layer="95" rot="R180" xref="yes"/>
-</segment>
-</net>
-<net name="+12V" class="0">
-<segment>
 <pinref part="I/O" gate="A" pin="18"/>
 <wire x1="60.96" y1="215.9" x2="71.12" y2="215.9" width="0.1524" layer="91"/>
 <label x="71.12" y="215.9" size="1.778" layer="95" xref="yes"/>
+</segment>
+</net>
+<net name="+12V" class="0">
+<segment>
+<pinref part="I/O" gate="A" pin="20"/>
+<wire x1="60.96" y1="213.36" x2="71.12" y2="213.36" width="0.1524" layer="91"/>
+<label x="81.28" y="213.36" size="1.778" layer="95" xref="yes"/>
 </segment>
 </net>
@@
 </segment>
 </net>
-<net name="PB14" class="0">
+<net name="USB_OTG_HS_DM" class="0">
 <segment>
 <pinref part="U$2" gate="G$1" pin="PB14"/>
 <wire x1="284.226" y1="88.138" x2="279.4" y2="88.138" width="0.1524" layer="91"/>
-<label x="265.684" y="88.138" size="1.778" layer="95"/>
+<label x="260.604" y="88.138" size="1.778" layer="95"/>
 <wire x1="279.4" y1="88.138" x2="265.684" y2="88.138" width="0.15" layer="91"/>
 </segment>
-</net>
-<net name="PB15" class="0">
+<segment>
+<pinref part="COM" gate="A" pin="13"/>
+<wire x1="53.34" y1="154.94" x2="43.18" y2="154.94" width="0.1524" layer="91"/>
+<label x="43.18" y="154.94" size="1.27" layer="95" rot="R180" xref="yes"/>
+</segment>
+</net>
+<net name="USB_OTG_HS_DP" class="0">
 <segment>
 <pinref part="U$2" gate="G$1" pin="PB15"/>
-<label x="265.684" y="85.598" size="1.778" layer="95"/>
+<label x="260.604" y="85.598" size="1.778" layer="95"/>
 <wire x1="284.226" y1="85.598" x2="265.684" y2="85.598" width="0.1524" layer="91"/>
 </segment>
-</net>
+<segment>
+<pinref part="COM" gate="A" pin="14"/>
+<wire x1="60.96" y1="154.94" x2="73.66" y2="154.94" width="0.1524" layer="91"/>
+<label x="73.66" y="154.94" size="1.27" layer="95" xref="yes"/>
+</segment>
+</net>

Commit message: First Draft
Completed routing of first draft for main board
Connections:
- removed net N$32: IC1.DSR, JP1.6
Changed lines of the file:
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@@
 <grid distance="0.1" unitdist="inch" unit="inch" style="dots" multiple="1" display="yes" altdistance="0.01" altunitdist="inch" altunit="inch"/>
 <layers>
-<layer number="1" name="Top" color="4" fill="1" visible="yes" active="no"/>
-<layer number="2" name="Route2" color="1" fill="3" visible="yes" active="no"/>
-<layer number="3" name="Route3" color="4" fill="3" visible="yes" active="no"/>
-<layer number="4" name="Route4" color="1" fill="4" visible="yes" active="no"/>
-<layer number="5" name="Route5" color="4" fill="4" visible="yes" active="no"/>
-<layer number="6" name="Route6" color="1" fill="8" visible="yes" active="no"/>
-<layer number="7" name="Route7" color="4" fill="8" visible="yes" active="no"/>
-<layer number="8" name="Route8" color="1" fill="2" visible="yes" active="no"/>
-<layer number="9" name="Route9" color="4" fill="2" visible="yes" active="no"/>
-<layer number="10" name="Route10" color="1" fill="7" visible="yes" active="no"/>
-<layer number="11" name="Route11" color="4" fill="7" visible="yes" active="no"/>
-<layer number="12" name="Route12" color="1" fill="5" visible="yes" active="no"/>
-<layer number="13" name="Route13" color="4" fill="5" visible="yes" active="no"/>
-<layer number="14" name="Route14" color="1" fill="6" visible="yes" active="no"/>
-<layer number="15" name="Route15" color="4" fill="6" visible="yes" active="no"/>
-<layer number="16" name="Bottom" color="1" fill="1" visible="yes" active="no"/>
-<layer number="17" name="Pads" color="2" fill="1" visible="yes" active="no"/>
-<layer number="18" name="Vias" color="2" fill="1" visible="yes" active="no"/>
-<layer number="19" name="Unrouted" color="6" fill="1" visible="yes" active="no"/>
-<layer number="20" name="Dimension" color="24" fill="1" visible="yes" active="no"/>
-<layer number="21" name="tPlace" color="7" fill="1" visible="yes" active="no"/>
-<layer number="22" name="bPlace" color="7" fill="1" visible="yes" active="no"/>
-<layer number="23" name="tOrigins" color="15" fill="1" visible="yes" active="no"/>
-<layer number="24" name="bOrigins" color="15" fill="1" visible="yes" active="no"/>
-<layer number="25" name="tNames" color="7" fill="1" visible="yes" active="no"/>
-<layer number="26" name="bNames" color="7" fill="1" visible="yes" active="no"/>
-<layer number="27" name="tValues" color="7" fill="1" visible="yes" active="no"/>
-<layer number="28" name="bValues" color="7" fill="1" visible="yes" active="no"/>
+<layer number="1" name="Top" color="4" fill="1" visible="no" active="no"/>
+<layer number="2" name="Route2" color="1" fill="3" visible="no" active="no"/>
+<layer number="3" name="Route3" color="4" fill="3" visible="no" active="no"/>
+<layer number="4" name="Route4" color="1" fill="4" visible="no" active="no"/>
+<layer number="5" name="Route5" color="4" fill="4" visible="no" active="no"/>
+<layer number="6" name="Route6" color="1" fill="8" visible="no" active="no"/>
+<layer number="7" name="Route7" color="4" fill="8" visible="no" active="no"/>
+<layer number="8" name="Route8" color="1" fill="2" visible="no" active="no"/>
+<layer number="9" name="Route9" color="4" fill="2" visible="no" active="no"/>
+<layer number="10" name="Route10" color="1" fill="7" visible="no" active="no"/>
+<layer number="11" name="Route11" color="4" fill="7" visible="no" active="no"/>
+<layer number="12" name="Route12" color="1" fill="5" visible="no" active="no"/>
+<layer number="13" name="Route13" color="4" fill="5" visible="no" active="no"/>
+<layer number="14" name="Route14" color="1" fill="6" visible="no" active="no"/>
+<layer number="15" name="Route15" color="4" fill="6" visible="no" active="no"/>
+<layer number="16" name="Bottom" color="1" fill="1" visible="no" active="no"/>
+<layer number="17" name="Pads" color="2" fill="1" visible="no" active="no"/>
+<layer number="18" name="Vias" color="2" fill="1" visible="no" active="no"/>
+<layer number="19" name="Unrouted" color="6" fill="1" visible="no" active="no"/>
+<layer number="20" name="Dimension" color="24" fill="1" visible="no" active="no"/>
+<layer number="21" name="tPlace" color="7" fill="1" visible="no" active="no"/>
+<layer number="22" name="bPlace" color="7" fill="1" visible="no" active="no"/>
+<layer number="23" name="tOrigins" color="15" fill="1" visible="no" active="no"/>
+<layer number="24" name="bOrigins" color="15" fill="1" visible="no" active="no"/>
+<layer number="25" name="tNames" color="7" fill="1" visible="no" active="no"/>
+<layer number="26" name="bNames" color="7" fill="1" visible="no" active="no"/>
+<layer number="27" name="tValues" color="7" fill="1" visible="no" active="no"/>
+<layer number="28" name="bValues" color="7" fill="1" visible="no" active="no"/>
 <layer number="29" name="tStop" color="7" fill="3" visible="no" active="no"/>
 <layer number="30" name="bStop" color="7" fill="6" visible="no" active="no"/>
@@
 <layer number="35" name="tGlue" color="7" fill="4" visible="no" active="no"/>
 <layer number="36" name="bGlue" color="7" fill="5" visible="no" active="no"/>
-<layer number="37" name="tTest" color="7" fill="1" visible="yes" active="no"/>
-<layer number="38" name="bTest" color="7" fill="1" visible="yes" active="no"/>
+<layer number="37" name="tTest" color="7" fill="1" visible="no" active="no"/>
+<layer number="38" name="bTest" color="7" fill="1" visible="no" active="no"/>
 <layer number="39" name="tKeepout" color="4" fill="11" visible="no" active="no"/>
 <layer number="40" name="bKeepout" color="1" fill="11" visible="no" active="no"/>
@@
 <layer number="44" name="Drills" color="7" fill="1" visible="no" active="no"/>
 <layer number="45" name="Holes" color="7" fill="1" visible="no" active="no"/>
-<layer number="46" name="Milling" color="3" fill="1" visible="yes" active="no"/>
-<layer number="47" name="Measures" color="7" fill="1" visible="yes" active="no"/>
-<layer number="48" name="Document" color="7" fill="1" visible="yes" active="no"/>
-<layer number="49" name="Reference" color="7" fill="1" visible="yes" active="no"/>
-<layer number="50" name="dxf" color="12" fill="1" visible="yes" active="no"/>
-<layer number="51" name="tDocu" color="7" fill="1" visible="yes" active="no"/>
-<layer number="52" name="bDocu" color="7" fill="1" visible="yes" active="no"/>
-<layer number="53" name="tGND_GNDA" color="7" fill="1" visible="yes" active="no"/>
-<layer number="54" name="bGND_GNDA" color="7" fill="1" visible="yes" active="no"/>
-<layer number="56" name="wert" color="7" fill="1" visible="yes" active="no"/>
-<layer number="57" name="tCAD" color="7" fill="1" visible="yes" active="no"/>
-<layer number="59" name="tCarbon" color="7" fill="1" visible="yes" active="no"/>
-<layer number="60" name="bCarbon" color="7" fill="1" visible="yes" active="no"/>
+<layer number="46" name="Milling" color="3" fill="1" visible="no" active="no"/>
+<layer number="47" name="Measures" color="7" fill="1" visible="no" active="no"/>
+<layer number="48" name="Document" color="7" fill="1" visible="no" active="no"/>
+<layer number="49" name="Reference" color="7" fill="1" visible="no" active="no"/>
+<layer number="50" name="dxf" color="12" fill="1" visible="no" active="no"/>
+<layer number="51" name="tDocu" color="7" fill="1" visible="no" active="no"/>
+<layer number="52" name="bDocu" color="7" fill="1" visible="no" active="no"/>
+<layer number="53" name="tGND_GNDA" color="7" fill="1" visible="no" active="no"/>
+<layer number="54" name="bGND_GNDA" color="7" fill="1" visible="no" active="no"/>
+<layer number="56" name="wert" color="7" fill="1" visible="no" active="no"/>
+<layer number="57" name="tCAD" color="7" fill="1" visible="no" active="no"/>
+<layer number="59" name="tCarbon" color="7" fill="1" visible="no" active="no"/>
+<layer number="60" name="bCarbon" color="7" fill="1" visible="no" active="no"/>
 <layer number="88" name="SimResults" color="9" fill="1" visible="yes" active="yes"/>
 <layer number="89" name="SimProbes" color="9" fill="1" visible="yes" active="yes"/>
@@
 </segment>
 </net>
-<net name="N$32" class="0">
-<segment>
-<pinref part="IC1" gate="G$1" pin="DSR"/>
-<wire x1="175.26" y1="73.66" x2="215.9" y2="73.66" width="0.1524" layer="91"/>
-<wire x1="215.9" y1="73.66" x2="215.9" y2="76.2" width="0.1524" layer="91"/>
-<pinref part="JP1" gate="A" pin="6"/>
-</segment>
-</net>

Commit message: First Revision
- Added 3 PIN terminal block for power
- Cleaned up tracks /rerouted
Parts:
- added X1: (no value), con-wago-500:W237-103
Connections:
- net +12V: now also X1-3.KL
- net GND: now also X1-2.KL
- net VIN: now also X1-1.KL
Changed lines of the file:
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@@
 <part name="RTS" library="jumper" library_urn="urn:adsk.eagle:library:252" deviceset="SJ" device="" package3d_urn="urn:adsk.eagle:package:15471/1"/>
 <part name="JP1" library="pinhead" library_urn="urn:adsk.eagle:library:325" deviceset="PINHD-1X6" device="" package3d_urn="urn:adsk.eagle:package:22472/2"/>
+<part name="X1" library="con-wago-500" library_urn="urn:adsk.eagle:library:195" deviceset="W237-103" device="" package3d_urn="urn:adsk.eagle:package:10691/1"/>
 </parts>
 <sheets>
@@
 <instance part="3V3" gate="G$1" x="66.802" y="-20.32" rot="MR0"/>
 <instance part="SUPPLY5" gate="+12V" x="66.802" y="-30.988" rot="R180"/>
+<instance part="X1" gate="-1" x="48.26" y="22.86"/>
+<instance part="X1" gate="-2" x="48.26" y="17.78"/>
+<instance part="X1" gate="-3" x="48.26" y="12.7"/>
 </instances>
 <busses>
@@
 <label x="15.24" y="17.78" size="1.778" layer="95" xref="yes"/>
 </segment>
+<segment>
+<pinref part="X1" gate="-2" pin="KL"/>
+<wire x1="53.34" y1="17.78" x2="60.96" y2="17.78" width="0.1524" layer="91"/>
+<label x="60.96" y="17.78" size="1.778" layer="95" xref="yes"/>
+</segment>
 </net>
 <net name="VIN" class="1">
@@
 <wire x1="5.08" y1="22.86" x2="15.24" y2="22.86" width="0.1524" layer="91"/>
 <label x="15.24" y="22.86" size="1.778" layer="95" xref="yes"/>
+</segment>
+<segment>
+<pinref part="X1" gate="-1" pin="KL"/>
+<wire x1="53.34" y1="22.86" x2="60.96" y2="22.86" width="0.1524" layer="91"/>
+<label x="60.96" y="22.86" size="1.778" layer="95" xref="yes"/>
 </segment>
 </net>
@@
 <wire x1="66.802" y1="-25.4" x2="66.802" y2="-28.448" width="0.1524" layer="91"/>
 </segment>
-</net>
+<segment>
+<pinref part="X1" gate="-3" pin="KL"/>
+<wire x1="53.34" y1="12.7" x2="60.96" y2="12.7" width="0.1524" layer="91"/>
+<label x="60.96" y="12.7" size="1.778" layer="95" xref="yes"/>
+</segment>
+</net>
