File: v1.1 - COM/schema_mpb_1_1_Serial.sch (EAGLE design)
At the start: 64 parts, among them U1 MAX232PTH, U2 MAX232PTH, U3 MAX232PTH

Commit message: RS232 Board
Routed tracks and added dimensions
Parts:
- removed C1, C10, C11, C12, C13, C14, C15, C2, C3, C4, C5, C6, C7, C8, C9: .1uF, rcl:C-EUC0805
- removed JP2: (no value), pinhead:PINHD-2X19
- removed JP3: (no value), pinhead:PINHD-2X14
- removed POWER: 8x1F-H8.5, SmartPrj:PINHD-1X8
- removed R10, R11, R19, R20: 10K, rcl:R-EU_R0805
- removed R12, R13, R21, R22: 4k7, rcl:R-EU_R0805
- removed R14, R23: 20R, rcl:R-EU_R0805
- removed R15, R16, R17, R18, R24, R25, R26, R27, R7, R8, R9: 1k, rcl:R-EU_R0805
- removed S1: SWITCH-MOMENTARY-2SMD-1101NE, SparkFun-Electromechanical:SWITCH-MOMENTARY-2SMD-1101NE
- removed T10, T11, T12, T9: (no value), semicon-smd-ipc:NPN-TRANSISTOR_SOT23
- removed U1, U2, U3: MAX232PTH, SparkFun-DigitalIC:MAX232PTH
- removed X3: (no value), con-wago-500:W237-6
- added C16, C17, C18, C19, C20, C21, C22, C23, C24, C25, C26, C27, C28, C29, C30: .1uF, rcl:C-EUC0603
- added H1, H2, H3, H4: MOUNT-PAD-ROUND3.2, holes:MOUNT-PAD-ROUND3.2
- added JP1: (no value), pinhead:PINHD-2X10
- added R28, R29, R37, R38, R46, R47: 10K, rcl:R-EU_R0603
- added R30, R31, R39, R40, R48, R49: 4k7, rcl:R-EU_R0603
- added R32, R41, R50: 20R, rcl:R-EU_R0603
- added R33, R34, R35, R36, R42, R43, R44, R45, R51, R52, R53, R54: 1k, rcl:R-EU_R0603
- added T13, T14, T17, T18, T19, T20, T21, T22, T23, T24: (no value), semicon-smd-ipc:NPN-TRANSISTOR_SOT23
- added U4, U5, U6: MAX232PTH, SparkFun-DigitalIC:MAX232PTH
- R1, R2: value 10K -> 1k; device rcl:R-EU_R0805 -> rcl:R-EU_R0603
- R3, R4: value 4k7 -> 1k; device rcl:R-EU_R0805 -> rcl:R-EU_R0603
- R5: value 20R -> 1k; device rcl:R-EU_R0805 -> rcl:R-EU_R0603
- R6: device rcl:R-EU_R0805 -> rcl:R-EU_R0603
- X1: device con-wago-500:W237-6 -> con-wago-508:W237-12P
- X2: device con-wago-500:W237-6 -> con-wago-508:W237-06P
Connections:
- removed net +12V: POWER.1
- removed net 3.3V: C12.2, C3.2, C7.2, POWER.4, R14.2, R15.1, R16.1, R17.1, R18.1, R23.2, R24.1, R25.1, R26.1, R27.1, R5.2, R6.1, R7.1, R8.1, R9.1, X1-6.KL, X2-6.KL, X3-6.KL
- removed net ADC0: JP2.1
- removed net ADC1: JP2.3
- removed net ADC12: JP2.25
- removed net ADC13: JP2.27
- removed net ADC14: JP2.29
- removed net ADC15: JP2.31
- removed net ADC2: JP2.5
- removed net ADC3: JP2.7
- removed net ADC4: JP2.9
- removed net ADC5: JP2.11
- removed net ADC6: JP2.13
- removed net ADC7: JP2.15
- removed net IO0: JP2.4
- removed net IO1: JP2.6
- removed net IO2: JP2.10
- removed net IO3: JP2.12
- removed net IO4: JP2.2
- removed net IO5: JP2.8
- removed net IO6: JP2.18
- removed net IO7: JP2.20
- removed net IO8: JP2.22
- removed net IO9: JP2.24
- removed net N$10: R17.2, T7.B
- removed net N$11: R18.2, T8.B
- removed net N$12: C15.2, U3.C1-
- removed net N$13: C15.1, U3.C1+
- removed net N$14: C14.2, U3.C2-
- removed net N$15: C6.2, U1.C1-
- removed net N$16: C6.1, U1.C1+
- removed net N$17: C5.2, U1.C2-
- removed net N$18: C5.1, U1.C2+
- removed net N$19: C4.1, U1.V-
- removed net N$20: C2.2, R5.1, U1.VCC
- removed net N$21: C3.1, U1.V+
- removed net N$22: R6.2, T1.B
- removed net N$23: R7.2, T2.B
- removed net N$24: R8.2, T3.B
- removed net N$25: R9.2, T4.B
- removed net N$26: C14.1, U3.C2+
- removed net N$27: C13.1, U3.V-
- removed net N$28: C11.2, R23.1, U3.VCC
- removed net N$29: C12.1, U3.V+
- removed net N$30: R24.2, T9.B
- removed net N$31: R25.2, T10.B
- removed net N$32: R26.2, T11.B
- removed net N$33: R27.2, T12.B
- removed net N$7: C7.1, U2.V+
- removed net N$8: R15.2, T5.B
- removed net N$9: R16.2, T6.B
- removed net PA0: JP2.33
- removed net PA1: JP2.35
- removed net PA2: JP2.37
- removed net PA3: JP3.28
- removed net PA4: JP3.26
- removed net PA5: JP3.24
- removed net PA6: JP3.22
- removed net PA7: JP3.20
- removed net PB0: JP2.26
- removed net PB1: JP2.28
- removed net PB2: JP2.30
- removed net PB3: JP2.32
- removed net PB4: JP2.34
- removed net PB5: JP2.36
- removed net PB6: JP2.38
- removed net PB7: JP3.27
- removed net PC0: JP3.3
- removed net PC1: JP3.1
- removed net PC2: JP3.2
- removed net PC3: JP3.4
- removed net PC4: JP3.6
- removed net PC5: JP3.8
- removed net PC6: JP3.10
- removed net PC7: JP3.12
- removed net PD7: JP3.9
- removed net PG0: JP3.7
- removed net PG1: JP3.5
- removed net PG2: JP3.18
- removed net PL2: JP3.25
- removed net PL3: JP3.23
- removed net PL4: JP3.21
- removed net PL5: JP3.19
- removed net R1IN_1: R4.2, T4.E, U1.R1IN
- removed net R1IN_1#: T4.C, X1-2.KL
- removed net R1IN_2: R13.2, T8.E, U2.R1IN
- removed net R1IN_2#: T8.C, X2-2.KL
- removed net R1IN_3: R22.2, T12.E, U3.R1IN
- removed net R1IN_3#: T12.C, X3-2.KL
- removed net R2IN_1: R3.2, T2.E, U1.R2IN
- removed net R2IN_1#: T2.C, X1-3.KL
- removed net R2IN_2: R12.2, T6.E, U2.R2IN
- removed net R2IN_2#: T6.C, X2-3.KL
- removed net R2IN_3: R21.2, T10.E, U3.R2IN
- removed net R2IN_3#: T10.C, X3-3.KL
- removed net R2OUT_3: U3.R2OUT
- removed net REG_5V: POWER.2, POWER.5
- removed net RESET: POWER.3, S1.1
- removed net SCL: JP3.17
- removed net SDA: JP3.15
- removed net T1OUT_1: T3.E, U1.T1OUT
- removed net T1OUT_1#: T3.C, X1-4.KL
- removed net T1OUT_2: T7.E, U2.T1OUT
- removed net T1OUT_2#: T7.C, X2-4.KL
- removed net T1OUT_3: T11.E, U3.T1OUT
- removed net T1OUT_3#: T11.C, X3-4.KL
- removed net T2IN_3: R20.2, U3.T2IN
- removed net T2OUT_1: T1.E, U1.T2OUT
- removed net T2OUT_1#: T1.C, X1-5.KL
- removed net T2OUT_2: T5.E, U2.T2OUT
- removed net T2OUT_2#: T5.C, X2-5.KL
- removed net T2OUT_3: T9.E, U3.T2OUT
- removed net T2OUT_3#: T9.C, X3-5.KL
- removed net VIN: POWER.8
- new net +3V3: C17.2, C22.2, C27.2, JP1.19, JP1.20, R1.1, R2.1, R3.1, R32.2, R33.1, R34.1, R35.1, R36.1, R4.1, R41.2, R42.1, R43.1, R44.1, R45.1, R5.1, R50.2, R51.1, R52.1, R53.1, R54.1, R6.1
- new net +5V: JP1.15, JP1.16
- new net GND1: T8.C, X1-3.KL
- new net GND2: T7.C, X1-6.KL
- new net GND3: T6.C, X1-9.KL
- new net GND4: T5.C, X1-12.KL
- new net GND5: T4.C, X2-3.KL
- new net GND6: T3.C, X2-6.KL
- new net N$34: C20.2, U4.C1-
- new net N$35: C20.1, U4.C1+
- new net N$36: C19.2, U4.C2-
- new net N$37: C19.1, U4.C2+
- new net N$38: C18.1, U4.V-
- new net N$39: C16.2, R32.1, U4.VCC
- new net N$40: C17.1, U4.V+
- new net N$41: R33.2, T13.B
- new net N$42: R34.2, T14.B
- new net N$43: R35.2, T1.B
- new net N$44: R36.2, T2.B
- new net N$45: C25.2, U5.C1-
- new net N$46: C25.1, U5.C1+
- new net N$47: C24.2, U5.C2-
- new net N$48: C24.1, U5.C2+
- new net N$49: C23.1, U5.V-
- new net N$50: C21.2, R41.1, U5.VCC
- new net N$51: C22.1, U5.V+
- new net N$52: R42.2, T17.B
- new net N$53: R43.2, T18.B
- new net N$54: R44.2, T19.B
- new net N$55: R45.2, T20.B
- new net N$56: C30.2, U6.C1-
- new net N$57: C30.1, U6.C1+
- new net N$58: C29.2, U6.C2-
- new net N$59: C29.1, U6.C2+
- new net N$60: C28.1, U6.V-
- new net N$61: C26.2, R50.1, U6.VCC
- new net N$62: C27.1, U6.V+
- new net N$63: R51.2, T21.B
- new net N$64: R52.2, T22.B
- new net N$65: R53.2, T23.B
- new net N$66: R54.2, T24.B
- new net RX1: JP1.1, U4.R1OUT
- new net RX2: JP1.3, U4.R2OUT
- new net RX3: JP1.5, U5.R1OUT
- new net RX4: JP1.7, U5.R2OUT
- new net RX5: JP1.9, U6.R1OUT
- new net RX6: JP1.11, U6.R2OUT
- new net RXD1#: T2.C, X1-2.KL
- new net RXD2#: T14.C, X1-5.KL
- new net RXD3#: T20.C, X1-8.KL
- new net RXD4#: T18.C, X1-11.KL
- new net RXD5#: T24.C, X2-2.KL
- new net RXD6: R48.2, T22.E, U6.R2IN
- new net RXD6#: T22.C, X2-5.KL
- new net TX1: JP1.2, R28.2, U4.T1IN
- new net TX2: JP1.4, R29.2, U4.T2IN
- new net TX3: JP1.6, R37.2, U5.T1IN
- new net TX4: JP1.8, R38.2, U5.T2IN
- new net TX5: JP1.10, R46.2, U6.T1IN
- new net TX6: JP1.12, R47.2, U6.T2IN
- new net TXD1#: T1.C, X1-1.KL
- new net TXD2#: T13.C, X1-4.KL
- new net TXD3#: T19.C, X1-7.KL
- new net TXD4#: T17.C, X1-10.KL
- new net TXD5#: T23.C, X2-1.KL
- new net TXD6: T21.E, U6.T2OUT
- new net TXD6#: T21.C, X2-4.KL
- net GND: now also C16.1, C18.2, C21.1, C23.2, C26.1, C28.2, JP1.13, JP1.14, JP1.17, JP1.18, R28.1, R29.1, R30.1, R31.1, R37.1, R38.1, R39.1, R40.1, R46.1, R47.1, R48.1, R49.1, T3.E, T4.E, T5.E, T6.E, T7.E, T8.E, U4.GND, U5.GND, U6.GND; no longer C1.1, C11.1, C13.2, C2.1, C4.2, C8.2, POWER.6, POWER.7, R1.1, R10.1, R11.1, R12.1, R13.1, R19.1, R2.1, R20.1, R21.1, R22.1, R3.1, R4.1, S1.2, U1.GND, U2.GND, U3.GND, X1-1.KL, X2-1.KL, X3-1.KL
- net N$1: now also R1.2, T3.B; no longer C10.2, U2.C1-
- net N$2: now also R2.2, T4.B; no longer C10.1, U2.C1+
- net N$3: now also R3.2, T5.B; no longer C9.2, U2.C2-
- net N$4: now also R4.2, T6.B; no longer C9.1, U2.C2+
- net N$5: now also R5.2, T7.B; no longer C8.1, U2.V-
- net N$6: now also R6.2, T8.B; no longer C1.2, R14.1, U2.VCC
- net RXD1: now also R31.2, T2.E, U4.R1IN; no longer JP3.13, U1.R1OUT
- net RXD2: now also R30.2, T14.E, U4.R2IN; no longer JP2.14, U1.R2OUT
- net RXD3: now also R40.2, T20.E, U5.R1IN; no longer JP3.14, U2.R1OUT
- net RXD4: now also R39.2, T18.E, U5.R2IN; no longer JP2.19, U2.R2OUT
- net RXD5: now also R49.2, T24.E, U6.R1IN; no longer JP2.23, U3.R1OUT
- net TXD1: now also T1.E, U4.T1OUT; no longer JP3.11, R1.2, U1.T1IN
- net TXD2: now also T13.E, U4.T2OUT; no longer JP2.16, R2.2, U1.T2IN
- net TXD3: now also T19.E, U5.T1OUT; no longer JP3.16, R10.2, U2.T1IN
- net TXD4: now also T17.E, U5.T2OUT; no longer JP2.17, R11.2, U2.T2IN
- net TXD5: now also T23.E, U6.T1OUT; no longer JP2.21, R19.2, U3.T1IN
Other:
- note removed: "2222A"
- note removed: "Pinout"
- moved on the sheet: R1, R2, R3, R4, R5, R6, T1, T2, T3, T4, T5, T6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
