File: v1.1 - COM board/schema_mpb_1_1_COM.sch (EAGLE design)
At the start: 0 parts

Commit message: Main board
- Rounded corners (2.54mm setting)
- Placed final mounting pad
Parts:
- added IC1: E73_2G4M04S, E73-2G4M04S:E73_2G4M04S
- added U1: ESP-WROOM-32, esp32:ESP-WROOM-32
