File: v1.1 - Main board/schema_mpb1_1.sch (EAGLE design)
At the start: 79 parts, among them IC1 CP2102, Q1 8M, Q2 32.768kHz, U1 NCP1117ST33T3G, U2 NCP1117ST50T3G, X2 PN61729-S, X5 POWERSUPPLY_DC21MMX

Commit message: Main board
- Tidy routes
Connections:
- net CAN1_RX: now also COM.6
- net CAN1_TX: no longer COM.6
Changed lines of the file:
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@@
 <wire x1="279.4" y1="138.938" x2="265.176" y2="138.938" width="0.15" layer="91"/>
+</segment>
+<segment>
+<pinref part="COM" gate="A" pin="6"/>
+<wire x1="60.96" y1="165.1" x2="73.66" y2="165.1" width="0.1524" layer="91"/>
+<label x="73.66" y="165.1" size="1.27" layer="95" xref="yes"/>
 </segment>
 </net>
@@
 <label x="43.18" y="165.1" size="1.27" layer="95" rot="R180" xref="yes"/>
 </segment>
-<segment>
-<pinref part="COM" gate="A" pin="6"/>
-<wire x1="60.96" y1="165.1" x2="73.66" y2="165.1" width="0.1524" layer="91"/>
-<label x="73.66" y="165.1" size="1.27" layer="95" xref="yes"/>
-</segment>
 </net>

Commit message: COM board
- Routed first version of Wireless COM board
Connections:
- net NRF_CE renamed NRF_TX
- net NRF_CS renamed NRF_RX
- net NRF_IRQ renamed PB8
- net NRF_MISO renamed PB4
- net NRF_MOSI renamed ESP_RX
- net NRF_SCK renamed ESP_TX
Other:
- moved on the sheet: B1, R4
Changed lines of the file:
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@@
 <instance part="Q2" gate="G$1" x="383.032" y="173.736"/>
 <instance part="Q1" gate="G$1" x="348.742" y="73.406"/>
-<instance part="B1" gate="G$1" x="239.268" y="118.618" rot="MR0"/>
-<instance part="SUPPLY4" gate="GND" x="239.268" y="104.648"/>
-<instance part="+3V1" gate="G$1" x="239.268" y="131.572" rot="MR0"/>
-<instance part="R4" gate="G$1" x="251.46" y="118.618"/>
+<instance part="B1" gate="G$1" x="224.028" y="118.618" rot="MR0"/>
+<instance part="SUPPLY4" gate="GND" x="224.028" y="104.648"/>
+<instance part="+3V1" gate="G$1" x="224.028" y="131.572" rot="MR0"/>
+<instance part="R4" gate="G$1" x="236.22" y="118.618"/>
 <instance part="B0" gate="G$1" x="224.536" y="234.95" rot="MR0"/>
 <instance part="SUPPLY7" gate="GND" x="224.536" y="225.806"/>
@@
 <segment>
 <pinref part="B1" gate="G$1" pin="3"/>
-<wire x1="239.268" y1="113.538" x2="239.268" y2="107.188" width="0.1524" layer="91"/>
+<wire x1="224.028" y1="113.538" x2="224.028" y2="107.188" width="0.1524" layer="91"/>
 <pinref part="SUPPLY4" gate="GND" pin="GND"/>
 </segment>
@@
 <segment>
 <pinref part="R4" gate="G$1" pin="2"/>
-<wire x1="256.54" y1="118.618" x2="261.366" y2="118.618" width="0.1524" layer="91"/>
-<wire x1="261.366" y1="118.872" x2="261.366" y2="118.618" width="0.1524" layer="91"/>
-<label x="261.366" y="118.618" size="1.778" layer="95" rot="R270" xref="yes"/>
+<wire x1="241.3" y1="118.618" x2="246.126" y2="118.618" width="0.1524" layer="91"/>
+<wire x1="246.126" y1="118.872" x2="246.126" y2="118.618" width="0.1524" layer="91"/>
+<label x="246.126" y="118.618" size="1.778" layer="95" rot="R270" xref="yes"/>
 </segment>
 </net>
@@
 <segment>
 <pinref part="B1" gate="G$1" pin="1"/>
-<wire x1="239.268" y1="123.698" x2="239.268" y2="128.778" width="0.1524" layer="91"/>
+<wire x1="224.028" y1="123.698" x2="224.028" y2="128.778" width="0.1524" layer="91"/>
 <pinref part="+3V1" gate="G$1" pin="+3V3"/>
-<wire x1="239.268" y1="123.698" x2="239.268" y2="129.032" width="0.1524" layer="91"/>
-<junction x="239.268" y="123.698"/>
+<wire x1="224.028" y1="123.698" x2="224.028" y2="129.032" width="0.1524" layer="91"/>
+<junction x="224.028" y="123.698"/>
 </segment>
 <segment>
@@
 </segment>
 </net>
-<net name="NRF_CE" class="0">
+<net name="NRF_TX" class="0">
 <segment>
 <pinref part="U$2" gate="G$1" pin="PB6"/>
@@
 </segment>
 </net>
-<net name="NRF_CS" class="0">
+<net name="NRF_RX" class="0">
 <segment>
 <pinref part="U$2" gate="G$1" pin="PB7"/>
@@
 </segment>
 </net>
-<net name="NRF_SCK" class="0">
+<net name="ESP_TX" class="0">
 <segment>
 <pinref part="U$2" gate="G$1" pin="PB3"/>
@@
 </segment>
 </net>
-<net name="NRF_MOSI" class="0">
+<net name="ESP_RX" class="0">
 <segment>
 <pinref part="U$2" gate="G$1" pin="PB5"/>
@@
 </segment>
 </net>
-<net name="NRF_MISO" class="0">
+<net name="PB4" class="0">
 <segment>
 <pinref part="U$2" gate="G$1" pin="PB4"/>
@@
 </segment>
 </net>
-<net name="NRF_IRQ" class="0">
+<net name="PB8" class="0">
 <segment>
 <pinref part="U$2" gate="G$1" pin="PB8"/>
@@
 <pinref part="B1" gate="G$1" pin="2"/>
 <pinref part="R4" gate="G$1" pin="1"/>
-<wire x1="244.348" y1="118.618" x2="246.38" y2="118.618" width="0.1524" layer="91"/>
-</segment>
-</net>
+<wire x1="229.108" y1="118.618" x2="231.14" y2="118.618" width="0.1524" layer="91"/>
+</segment>
+</net>

Commit message: Logos
Added Geviton Logo to designs
Changed lines of the file:
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@@
+</nets>
+</sheet>
+<sheet>
+<plain>
+</plain>
+<instances>
+</instances>
+<busses>
+</busses>
+<nets>
 </nets>
 </sheet>
